File: arcs_pwr_ctrl_conversion_fw/arcs_pwr_ctrl_conversion_fw.kicad_pcb (KiCad board)
At the start: 2 copper layers, 99 x 130 mm, 5 parts, among them J2 81100-560203-RB, J4 5747842-3

Commit message: Add Rev 1
Parts:
- removed BT1: 9V, Connector_PinHeader_2.54mm:PinHeader_1x02_P2.54mm_Vertical
- removed D1: 2V RED, LED_THT:LED_D1.8mm_W1.8mm_H2.4mm_Horizontal_O1.27mm_Z1.6mm
- removed R1: 470, Resistor_THT:R_Axial_DIN0414_L11.9mm_D4.5mm_P20.32mm_Horizontal
- added G***: LOGO, LOGO, F.Cu at (136.5, 126.5)
- added J3: 5747842-3, footprints:CONN25x1_5747842-3_TEC, F.Cu at (167.5, 66.9)
- moved J2 86.2 mm to (167.5, 125.9), turned to 90 degrees
- moved J1 76.3 mm to (142.0, 111.2), turned to 90 degrees
- renumbered J2 to J1, J4 to J2
Connections:
- J1 pad 100: CMB5-VDDP -> CMB1-VDDP
- J1 pad 22: CMB2-VDD -> CMB1-VDD
- J1 pad 23: CMB2-TEST -> CMB1-TEST
- J1 pad 24: CMB2-VDD -> CMB1-VDD
- J1 pad 25: CMB2-RST -> CMB1-RST
- J1 pad 26: CMB2-VDD -> CMB1-VDD
- J1 pad 27: CMB2-CS -> CMB1-CS
- J1 pad 28: CMB2-VDD -> CMB1-VDD
- J1 pad 29: CMB2-CLK -> CMB1-CLK
- J1 pad 30: CMB2-VDD -> CMB1-VDD
- J1 pad 32: CMB2-VDDP -> CMB1-VDDP
- J1 pad 34: CMB2-VDDP -> CMB1-VDDP
- J1 pad 36: CMB2-VDDP -> CMB1-VDDP
- J1 pad 38: CMB2-VDDP -> CMB1-VDDP
- J1 pad 40: CMB2-VDDP -> CMB1-VDDP
- J1 pad 42: CMB3-VDD -> CMB1-VDD
- J1 pad 43: CMB3-TEST -> CMB1-TEST
- J1 pad 44: CMB3-VDD -> CMB1-VDD
- J1 pad 45: CMB3-RST -> CMB1-RST
- J1 pad 46: CMB3-VDD -> CMB1-VDD
- J1 pad 47: CMB3-CS -> CMB1-CS
- J1 pad 48: CMB3-VDD -> CMB1-VDD
- J1 pad 49: CMB3-CLK -> CMB1-CLK
- J1 pad 50: CMB3-VDD -> CMB1-VDD
- J1 pad 52: CMB3-VDDP -> CMB1-VDDP
- J1 pad 54: CMB3-VDDP -> CMB1-VDDP
- J1 pad 56: CMB3-VDDP -> CMB1-VDDP
- J1 pad 58: CMB3-VDDP -> CMB1-VDDP
- J1 pad 60: CMB3-VDDP -> CMB1-VDDP
- J1 pad 62: CMB4-VDD -> CMB1-VDD
- J1 pad 63: CMB4-TEST -> CMB1-TEST
- J1 pad 64: CMB4-VDD -> CMB1-VDD
- J1 pad 65: CMB4-RST -> CMB1-RST
- J1 pad 66: CMB4-VDD -> CMB1-VDD
- J1 pad 67: CMB4-CS -> CMB1-CS
- J1 pad 68: CMB4-VDD -> CMB1-VDD
- J1 pad 69: CMB4-CLK -> CMB1-CLK
- J1 pad 70: CMB4-VDD -> CMB1-VDD
- J1 pad 72: CMB4-VDDP -> CMB1-VDDP
- J1 pad 74: CMB4-VDDP -> CMB1-VDDP
- J1 pad 76: CMB4-VDDP -> CMB1-VDDP
- J1 pad 78: CMB4-VDDP -> CMB1-VDDP
- J1 pad 80: CMB4-VDDP -> CMB1-VDDP
- J1 pad 82: CMB5-VDD -> CMB1-VDD
- J1 pad 83: CMB5-TEST -> CMB1-TEST
- J1 pad 84: CMB5-VDD -> CMB1-VDD
- J1 pad 85: CMB5-RST -> CMB1-RST
- J1 pad 86: CMB5-VDD -> CMB1-VDD
- J1 pad 87: CMB5-CS -> CMB1-CS
- J1 pad 88: CMB5-VDD -> CMB1-VDD
- J1 pad 89: CMB5-CLK -> CMB1-CLK
- J1 pad 90: CMB5-VDD -> CMB1-VDD
- J1 pad 92: CMB5-VDDP -> CMB1-VDDP
- J1 pad 94: CMB5-VDDP -> CMB1-VDDP
- J1 pad 96: CMB5-VDDP -> CMB1-VDDP
- J1 pad 98: CMB5-VDDP -> CMB1-VDDP
- J2 pad 10: CMB2-VDD-S -> CMB1-VDD-S
- J2 pad 11: CMB2-SDO-3 -> CMB1-SDO-3
- J2 pad 12: CMB2-SDI-1 -> CMB1-SDI-1
- J2 pad 13: CMB2-VDDP-S -> CMB1-VDDP-S
- J2 pad 14: unconnected-(J4-Pad14) -> CMB2-VDD-S
- J2 pad 15: unconnected-(J4-Pad15) -> CMB2-SDO-3
- J2 pad 16: unconnected-(J4-Pad16) -> CMB2-SDI-1
- J2 pad 17: unconnected-(J4-Pad17) -> CMB2-VDDP-S
- J2 pad 18: unconnected-(J4-Pad18) -> CMB3-VDD-S
- J2 pad 19: unconnected-(J4-Pad19) -> CMB3-SDO-3
- J2 pad 20: unconnected-(J4-Pad20) -> CMB3-SDI-1
- J2 pad 21: unconnected-(J4-Pad21) -> CMB3-VDDP-S
- J2 pad 22: unconnected-(J4-Pad22) -> CMB4-VDD-S
- J2 pad 23: unconnected-(J4-Pad23) -> CMB4-SDO-3
- J2 pad 24: unconnected-(J4-Pad24) -> CMB4-SDI-1
- J2 pad 25: unconnected-(J4-Pad25) -> CMB4-VDDP-S
- J2 pad 4: CMB1-VDDP -> CMB1-VDD
- J2 pad 5: CMB1-VDDP -> CMB1-VDD
- J2 pad 6: CMB1-VDD-S -> CMB1-VDD
- J2 pad 7: CMB1-SDO-3 -> CMB1-VDD
- J2 pad 8: CMB1-SDI-1 -> CMB1-VDD
- J2 pad 9: CMB1-VDDP-S -> CMB1-VDD
Routing:
- net CMB1-CLK: track 0.00 -> 192.9 mm
- net CMB1-RST: track 0.00 -> 181.0 mm
- net CMB1-CS: track 0.00 -> 173.3 mm
- net CMB1-TEST: track 0.00 -> 167.2 mm
- net CMB1-VDD: track 66.6 -> 128.8 mm
- net CMB1-VDDP: track 84.9 -> 132.5 mm
- net CMB4-SDI-1: track 0.00 -> 44.6 mm
- net CMB4-VDDP-S: track 0.00 -> 41.8 mm
- net CMB4-SDO-3: track 0.00 -> 40.6 mm
- net CMB3-SDI-1: track 0.00 -> 38.7 mm
- net CMB4-VDD-S: track 0.00 -> 38.2 mm
- net CMB5-VDD-S: track 0.00 -> 37.6 mm
- net CMB5-SDI-1: track 0.00 -> 36.1 mm
- net CMB2-SDI-1: track 0.00 -> 35.7 mm
- net CMB3-VDDP-S: track 0.00 -> 35.3 mm
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Other:
- board size 99 x 130 mm -> 58.5 x 119.5 mm
- copper layers 2 -> 4
- board text added: "ArCS Power Control Adapter Board Rev 1"
