File: arcs_pwr_ctrl_conversion_fw/arcs_pwr_ctrl_conversion_fw.kicad_sch (KiCad schematic)
At the start: 5 parts, among them J2 81100-560203-RB, J4 5747842-3

Commit message: Add Rev 1
Parts:
- removed BT1: 9V, Connector_PinHeader_2.54mm:PinHeader_1x02_P2.54mm_Vertical, symbol Device:Battery
- removed D1: 2V RED, LED_THT:LED_D1.8mm_W1.8mm_H2.4mm_Horizontal_O1.27mm_Z1.6mm, symbol Device:LED
- removed R1: 470, Resistor_THT:R_Axial_DIN0414_L11.9mm_D4.5mm_P20.32mm_Horizontal, symbol Device:R
- added J3: 5747842-3, footprints:CONN25x1_5747842-3_TEC, symbol 5747842-3:5747842-3
- renumbered J2 to J1, J4 to J2
Connections:
- net CMB2-CLK is gone; now on net CMB1-CLK: J1.29
- net CMB2-CS is gone; now on net CMB1-CS: J1.27
- net CMB2-RST is gone; now on net CMB1-RST: J1.25
- net CMB2-TEST is gone; now on net CMB1-TEST: J1.23
- net CMB2-VDD is gone; now on net CMB1-VDD: J1.22, J1.24, J1.26, J1.28, J1.30
- net CMB2-VDDP is gone; now on net CMB1-VDDP: J1.32, J1.34, J1.36, J1.38, J1.40
- net CMB3-CLK is gone; now on net CMB1-CLK: J1.49
- net CMB3-CS is gone; now on net CMB1-CS: J1.47
- net CMB3-RST is gone; now on net CMB1-RST: J1.45
- net CMB3-TEST is gone; now on net CMB1-TEST: J1.43
- net CMB3-VDD is gone; now on net CMB1-VDD: J1.42, J1.44, J1.46, J1.48, J1.50
- net CMB3-VDDP is gone; now on net CMB1-VDDP: J1.52, J1.54, J1.56, J1.58, J1.60
- net CMB4-CLK is gone; now on net CMB1-CLK: J1.69
- net CMB4-CS is gone; now on net CMB1-CS: J1.67
- net CMB4-RST is gone; now on net CMB1-RST: J1.65
- net CMB4-TEST is gone; now on net CMB1-TEST: J1.63
- net CMB4-VDD is gone; now on net CMB1-VDD: J1.62, J1.64, J1.66, J1.68, J1.70
- net CMB4-VDDP is gone; now on net CMB1-VDDP: J1.72, J1.74, J1.76, J1.78, J1.80
- net CMB5-CLK is gone; now on net CMB1-CLK: J1.89
- net CMB5-CS is gone; now on net CMB1-CS: J1.87
- net CMB5-RST is gone; now on net CMB1-RST: J1.85
- net CMB5-TEST is gone; now on net CMB1-TEST: J1.83
- net CMB5-VDD is gone; now on net CMB1-VDD: J1.82, J1.84, J1.86, J1.88, J1.90
- net CMB5-VDDP is gone; now on net CMB1-VDDP: J1.100, J1.92, J1.94, J1.96, J1.98
- net CMB1-CLK: now also J3.19, J3.20, J3.21
- net CMB1-CS: now also J3.16, J3.17, J3.18
- net CMB1-RST: now also J3.13, J3.14, J3.15
- net CMB1-SDI-1: now also J2.12; no longer J2.8
- net CMB1-SDO-3: now also J2.11; no longer J2.7
- net CMB1-TEST: now also J3.10, J3.11, J3.12
- net CMB1-VDD: now also J2.4, J2.5, J2.6, J2.7, J2.8, J2.9
- net CMB1-VDD-S: now also J2.10; no longer J2.6
- net CMB1-VDDP: now also J3.1, J3.2, J3.3, J3.4, J3.5, J3.6, J3.7, J3.8, J3.9; no longer J2.4, J2.5
- net CMB1-VDDP-S: now also J2.13; no longer J2.9
- net CMB2-SDI-1: now also J2.16; no longer J2.12
- net CMB2-SDO-3: now also J2.15; no longer J2.11
- net CMB2-VDD-S: now also J2.14; no longer J2.10
- net CMB2-VDDP-S: now also J2.17; no longer J2.13
- net CMB3-SDI-1: now also J2.20
- net CMB3-SDO-3: now also J2.19
- net CMB3-VDD-S: now also J2.18
- net CMB3-VDDP-S: now also J2.21
- net CMB4-SDI-1: now also J2.24
- net CMB4-SDO-3: now also J2.23
- net CMB4-VDD-S: now also J2.22
- net CMB4-VDDP-S: now also J2.25
- net CMB5-SDI-1: now also J3.24
- net CMB5-SDO-3: now also J3.23
- net CMB5-VDD-S: now also J3.22
- net CMB5-VDDP-S: now also J3.25
Other:
- company: (none) -> Fermilab
- title: (none) -> ArCS Power Control Adapter Board
- moved on the sheet: J2
